File: docs/kicad_weather_station/kicad_weather_station.kicad_sch (KiCad schematic)
At the start: 3 parts, among them U1 DHT11

Commit message: Creating docs
Parts:
- DS1: footprint Display:WC1602A -> RowBasedDisplay:WC1602A
Changed lines of the file:
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@@
       (effects (font (size 1.27 1.27)) (justify left))
     )
-    (property "Footprint" "Display:WC1602A" (at 132.08 78.74 0)
+    (property "Footprint" "RowBasedDisplay:WC1602A" (at 132.08 78.74 0)
       (effects (font (size 1.27 1.27) italic) hide)
     )

Commit message: Fisrt creating how i think the implementations will be defined
Parts:
- DS1: footprint RowBasedDisplay:WC1602A -> TextBasedDisplay:WC1602A
Changed lines of the file:
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@@
       (effects (font (size 1.27 1.27)) (justify left))
     )
-    (property "Footprint" "RowBasedDisplay:WC1602A" (at 132.08 78.74 0)
+    (property "Footprint" "TextBasedDisplay:WC1602A" (at 132.08 78.74 0)
       (effects (font (size 1.27 1.27) italic) hide)
     )
